File: Toaplan2/Raizing/RA9704/ra9704-kicad/audio-dac-sfx-roms.kicad_sch (KiCad schematic)
At the start: 6 parts, among them U823 YM2151, U827 27C040, U828 M6295, U829 27C040, U830 M6295

Commit message: feature(ra9704): rev 002
Changed lines of the file:
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@@
 	(title_block
 		(title "RA9704, Audio DAC and Sound Effect ROMs")
-		(date "2024-12-29")
+		(date "2024-12-30")
 		(rev "002")
 		(company "Coin-Op Collection")
@@
 	)
 	(bus_entry
+		(at 43.18 58.42)
+		(size 2.54 2.54)
+		(stroke
+			(width 0)
+			(type default)
+		)
+	)
+	(bus_entry
 		(at 110.49 165.1)
 		(size -2.54 -2.54)
@@
 		)
 	)
+	(bus
+		(pts
+			(xy 36.83 58.42) (xy 43.18 58.42)
+		)
+		(stroke
+			(width 0)
+			(type default)
+		)
+	)
 	(wire
 		(pts
@@
 		)
 	)
-	(wire
-		(pts
-			(xy 331.47 93.98) (xy 341.63 93.98)
-		)
-		(stroke
-			(width 0)
-			(type default)
-		)
-	)
 	(bus
 		(pts
@@
 		)
 	)
+	(wire
+		(pts
+			(xy 45.72 60.96) (xy 67.31 60.96)
+		)
+		(stroke
+			(width 0)
+			(type default)
+		)
+	)
 	(bus
 		(pts
@@
 		)
 	)
-	(label "SFX1_A[0..7]"
+	(label "SFX1_A[0..18]"
 		(at 176.53 125.73 90)
 		(fields_autoplaced yes)
@@
 		)
 	)
-	(label "SFX2_A[0..7]"
+	(label "SFX2_A[0..18]"
 		(at 328.93 125.73 90)
 		(fields_autoplaced yes)
@@
 		)
 	)
-	(label "SFX2_A11"
-		(at 331.47 71.12 0)
+	(label "SBUS_A0"
+		(at 45.72 60.96 0)
 		(fields_autoplaced yes)
 		(effects
@@
 		)
 	)
-	(label "YM2151_D7"
-		(at 110.49 35.56 0)
+	(label "SFX2_A11"
+		(at 331.47 71.12 0)
 		(fields_autoplaced yes)
 		(effects
@@
 		)
 	)
-	(label "SFX1_A11"
-		(at 179.07 71.12 0)
+	(label "YM2151_D7"
+		(at 110.49 35.56 0)
 		(fields_autoplaced yes)
 		(effects
@@
 		)
 	)
-	(label "YM2151_D[0..7]"
-		(at 107.95 125.73 90)
+	(label "SFX1_A11"
+		(at 179.07 71.12 0)
 		(fields_autoplaced yes)
 		(effects
@@
 		)
 	)
-	(label "SFX2_VPP"
-		(at 331.47 93.98 0)
+	(label "YM2151_D[0..7]"
+		(at 107.95 125.73 90)
 		(fields_autoplaced yes)
 		(effects
@@
 		)
 	)
-	(hierarchical_label "SFX2_A[0..7]"
+	(hierarchical_label "SFX2_A[0..18]"
 		(shape bidirectional)
 		(at 334.01 128.27 0)
@@
 	)
 	(hierarchical_label "ADPCM1_DAO"
-		(shape input)
+		(shape output)
 		(at 316.23 195.58 0)
 		(fields_autoplaced yes)
@@
 		)
 	)
-	(hierarchical_label "SFX1_A[0..7]"
+	(hierarchical_label "SFX1_A[0..18]"
 		(shape bidirectional)
 		(at 181.61 128.27 0)
@@
 		)
 	)
-	(hierarchical_label "SBUS_A0"
+	(hierarchical_label "SCPU_~{WR}"
 		(shape input)
-		(at 67.31 60.96 180)
+		(at 316.23 200.66 0)
 		(fields_autoplaced yes)
 		(effects
@@
 				(size 1.27 1.27)
 			)
-			(justify right)
+			(justify left)
 		)
 	)
-	(hierarchical_label "SCPU_~{WR}"
+	(hierarchical_label "ADPCM_XT"
 		(shape input)
-		(at 316.23 200.66 0)
+		(at 316.23 205.74 0)
 		(fields_autoplaced yes)
 		(effects
@@
 		)
 	)
-	(hierarchical_label "ADPCM_XT"
+	(hierarchical_label "SBUS_A[0..15]"
 		(shape input)
-		(at 316.23 205.74 0)
+		(at 36.83 58.42 180)
 		(fields_autoplaced yes)
 		(effects
@@
 				(size 1.27 1.27)
 			)
-			(justify left)
+			(justify right)
 		)
 	)
@@
 	)
 	(hierarchical_label "ADPCM2_DAO"
-		(shape input)
+		(shape output)
 		(at 163.83 195.58 0)
 		(fields_autoplaced yes)
@@
 		)
 	)
+	(hierarchical_label "SFX2_VPP"
+		(shape input)
+		(at 341.63 93.98 180)
+		(fields_autoplaced yes)
+		(effects
+			(font
+				(size 1.27 1.27)
+			)
+			(justify right)
+		)
+	)
