File: Toaplan2/Raizing/RA9704/ra9704-kicad/gcu-and-gcu_v-ram.kicad_sch (KiCad schematic)
At the start: 6 parts, among them U125 74HC245, U126 74HC245, U42 GP9001, U46 TMS45160DZ, U47 TMS45160DZ

Commit message: feature(ra9704): rev 002
Changed lines of the file:
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@@
 	(title_block
 		(title "RA9704, GCU and GCU_V RAM")
-		(date "2024-12-29")
+		(date "2024-12-30")
 		(rev "002")
 		(company "Coin-Op Collection")
@@
 		)
 	)
+	(wire
+		(pts
+			(xy 182.88 40.64) (xy 182.88 67.31)
+		)
+		(stroke
+			(width 0)
+			(type default)
+		)
+	)
 	(bus
 		(pts
@@
 	(wire
 		(pts
+			(xy 170.18 40.64) (xy 170.18 67.31)
+		)
+		(stroke
+			(width 0)
+			(type default)
+		)
+	)
+	(wire
+		(pts
 			(xy 373.38 194.31) (xy 383.54 194.31)
 		)
@@
 		)
 	)
-	(wire
-		(pts
-			(xy 170.18 55.88) (xy 170.18 67.31)
-		)
-		(stroke
-			(width 0)
-			(type default)
-		)
-	)
 	(bus
 		(pts
@@
 	(wire
 		(pts
-			(xy 347.98 82.55) (xy 359.41 82.55)
+			(xy 175.26 40.64) (xy 175.26 67.31)
 		)
 		(stroke
@@
 	(wire
 		(pts
-			(xy 233.68 171.45) (xy 245.11 171.45)
+			(xy 347.98 82.55) (xy 359.41 82.55)
 		)
 		(stroke
@@
 	(wire
 		(pts
-			(xy 137.16 229.87) (xy 137.16 217.17)
+			(xy 233.68 171.45) (xy 245.11 171.45)
 		)
 		(stroke
@@
 	(wire
 		(pts
-			(xy 359.41 54.61) (xy 347.98 54.61)
+			(xy 137.16 229.87) (xy 137.16 217.17)
 		)
 		(stroke
@@
 	(wire
 		(pts
-			(xy 185.42 55.88) (xy 185.42 67.31)
+			(xy 359.41 54.61) (xy 347.98 54.61)
 		)
 		(stroke
@@
 	(wire
 		(pts
-			(xy 180.34 55.88) (xy 180.34 67.31)
+			(xy 245.11 85.09) (xy 233.68 85.09)
 		)
 		(stroke
@@
 	(wire
 		(pts
-			(xy 245.11 85.09) (xy 233.68 85.09)
+			(xy 180.34 40.64) (xy 180.34 67.31)
 		)
 		(stroke
@@
 		)
 	)
+	(wire
+		(pts
+			(xy 177.8 40.64) (xy 177.8 67.31)
+		)
+		(stroke
+			(width 0)
+			(type default)
+		)
+	)
 	(bus
 		(pts
@@
 	(wire
 		(pts
-			(xy 167.64 54.61) (xy 167.64 67.31)
-		)
-		(stroke
-			(width 0)
-			(type default)
-		)
-	)
-	(wire
-		(pts
 			(xy 308.61 191.77) (xy 320.04 191.77)
 		)
@@
 	(wire
 		(pts
-			(xy 182.88 55.88) (xy 182.88 67.31)
-		)
-		(stroke
-			(width 0)
-			(type default)
-		)
-	)
-	(wire
-		(pts
 			(xy 373.38 186.69) (xy 383.54 186.69)
 		)
@@
 		)
 	)
-	(wire
-		(pts
-			(xy 177.8 55.88) (xy 177.8 67.31)
-		)
-		(stroke
-			(width 0)
-			(type default)
-		)
-	)
 	(bus
 		(pts
@@
 	(wire
 		(pts
-			(xy 187.96 55.88) (xy 187.96 67.31)
+			(xy 187.96 40.64) (xy 187.96 67.31)
 		)
 		(stroke
@@
 		)
 	)
-	(wire
-		(pts
-			(xy 175.26 55.88) (xy 175.26 67.31)
-		)
-		(stroke
-			(width 0)
-			(type default)
-		)
-	)
 	(bus
 		(pts
@@
 	(wire
 		(pts
+			(xy 185.42 40.64) (xy 185.42 67.31)
+		)
+		(stroke
+			(width 0)
+			(type default)
+		)
+	)
+	(wire
+		(pts
 			(xy 44.45 190.5) (xy 57.15 190.5)
 		)
@@
 	(wire
 		(pts
-			(xy 172.72 55.88) (xy 172.72 67.31)
+			(xy 172.72 40.64) (xy 172.72 67.31)
 		)
 		(stroke
@@
 	)
 	(label "GCU_V1_WE"
-		(at 170.18 67.31 90)
+		(at 170.18 53.34 90)
 		(fields_autoplaced yes)
 		(effects
@@
 	)
 	(label "GCU_V0_OE"
-		(at 182.88 67.31 90)
+		(at 182.88 53.34 90)
 		(fields_autoplaced yes)
 		(effects
@@
 		)
 	)
-	(label "GCU_OSCCLK"
-		(at 167.64 67.31 90)
-		(fields_autoplaced yes)
-		(effects
-			(font
-				(size 1.27 1.27)
-			)
-			(justify left bottom)
-		)
-	)
 	(label "GCU_V1D10"
 		(at 387.35 77.47 0)
@@
 		)
 	)
+	(label "GCU_D[0..15]"
+		(at 322.58 226.06 90)
+		(fields_autoplaced yes)
+		(effects
+			(font
+				(size 1.27 1.27)
+			)
+			(justify left bottom)
+		)
+	)
 	(label "GCU_V0D11"
 		(at 317.5 80.01 0)
@@
 		)
 	)
+	(label "GCU_OUT[0..10]"
+		(at 271.78 151.13 0)
+		(fields_autoplaced yes)
+		(effects
+			(font
+				(size 1.27 1.27)
+			)
+			(justify left bottom)
+		)
+	)
 	(label "GCU_FRA16"
 		(at 68.58 229.87 90)
@@
 		)
 	)
+	(label "MBUS_D[0..15]"
+		(at 271.78 160.02 0)
+		(fields_autoplaced yes)
+		(effects
+			(font
+				(size 1.27 1.27)
+			)
+			(justify left bottom)
+		)
+	)
 	(label "GCU_FMA3"
 		(at 91.44 229.87 90)
@@
 	)
 	(label "GCU_V0_WE"
-		(at 180.34 67.31 90)
+		(at 180.34 53.34 90)
 		(fields_autoplaced yes)
 		(effects
@@
 		)
 	)
+	(label "GCU_OUT[0..10]"
+		(at 335.28 151.13 0)
+		(fields_autoplaced yes)
+		(effects
+			(font
+				(size 1.27 1.27)
+			)
+			(justify left bottom)
+		)
+	)
 	(label "GCU_V0_OE"
 		(at 278.13 87.63 0)
@@
 		)
 	)
+	(label "MBUS_D[0..15]"
+		(at 334.01 175.26 90)
+		(fields_autoplaced yes)
+		(effects
+			(font
+				(size 1.27 1.27)
+			)
+			(justify left bottom)
+		)
+	)
 	(label "GCU_V0A[0..8]"
 		(at 275.59 52.07 90)
@@
 	)
 	(label "GCU_V0_CAS"
-		(at 187.96 67.31 90)
+		(at 187.96 53.34 90)
 		(fields_autoplaced yes)
 		(effects
@@
 	)
 	(label "GCU_V0_RAS"
-		(at 185.42 67.31 90)
+		(at 185.42 53.34 90)
 		(fields_autoplaced yes)
 		(effects
@@
 	)
 	(label "GCU_V0_RAS"
-		(at 177.8 67.31 90)
+		(at 177.8 53.34 90)
 		(fields_autoplaced yes)
 		(effects
@@
 	)
 	(label "GCU_V0_CAS"
-		(at 175.26 67.31 90)
+		(at 175.26 53.34 90)
 		(fields_autoplaced yes)
 		(effects
@@
 		)
 	)
+	(label "GCU_D[0..15]"
+		(at 386.08 226.06 90)
+		(fields_autoplaced yes)
+		(effects
+			(font
+				(size 1.27 1.27)
+			)
+			(justify left bottom)
+		)
+	)
 	(label "GCU_FRD27"
 		(at 44.45 149.86 0)
@@
 	)
 	(label "GCU_V1_OE"
-		(at 172.72 67.31 90)
+		(at 172.72 53.34 90)
 		(fields_autoplaced yes)
 		(effects
@@
 		)
 	)
+	(label "GCU_D[0..15]"
+		(at 248.92 227.33 0)
+		(fields_autoplaced yes)
+		(effects
+			(font
+				(size 1.27 1.27)
+			)
+			(justify left bottom)
+		)
+	)
 	(label "GCU_FRA10"
 		(at 44.45 190.5 0)
@@
 		)
 	)
+	(hierarchical_label "GCU_OSCCLK"
+		(shape input)
+		(at 167.64 67.31 90)
+		(fields_autoplaced yes)
+		(effects
+			(font
+				(size 1.27 1.27)
+			)
+			(justify left)
+		)
+	)
