File: Toaplan2/Raizing/RA9704/ra9704-kicad/gcu-and-gcu_v-ram.kicad_sch (KiCad schematic)
At the start: 6 parts, among them U125 74HC245, U126 74HC245, U42 GP9001, U46 TMS45160DZ, U47 TMS45160DZ

Commit message: fix(ra9704): Add Os as a proxy for 0s in all reference designators
RA9704 has reference designators such that each number has a preceding zero (e.g. RA076, U074, etc.). This causes a bug in KiCAD.

This is 'fixed' by using the 'O' (the letter 'Oh') character instead.

For more info, see the following issue on the KiCAD Gitlab repo

https://gitlab.com/kicad/code/kicad/-/issues/19229
Parts:
- renumbered RA41 to RA041, U125 to UO125, U126 to UO126, U42 to UO42, U46 to UO46, U47 to UO47
Connections:
- net U46_DQ12 renamed UO46_DQ12
- net U46_DQ13 renamed UO46_DQ13
- net U46_DQ14 renamed UO46_DQ14
- net U46_DQ15 renamed UO46_DQ15
- net U47_DQ12 renamed UO47_DQ12
- net U47_DQ13 renamed UO47_DQ13
- net U47_DQ14 renamed UO47_DQ14
- net U47_DQ15 renamed UO47_DQ15
Changed lines of the file:
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@@
 		)
 	)
-	(label "U46_DQ12"
+	(label "UO46_DQ12"
 		(at 334.01 125.73 0)
 		(fields_autoplaced yes)
@@
 		)
 	)
-	(label "U47_DQ12"
+	(label "UO47_DQ12"
 		(at 317.5 82.55 0)
 		(fields_autoplaced yes)
@@
 		)
 	)
-	(label "U47_DQ13"
+	(label "UO47_DQ13"
 		(at 334.01 133.35 0)
 		(fields_autoplaced yes)
@@
 		)
 	)
-	(label "U47_DQ12"
+	(label "UO47_DQ12"
 		(at 334.01 135.89 0)
 		(fields_autoplaced yes)
@@
 		)
 	)
-	(label "U46_DQ12"
+	(label "UO46_DQ12"
 		(at 387.35 82.55 0)
 		(fields_autoplaced yes)
@@
 		)
 	)
-	(label "U46_DQ14"
+	(label "UO46_DQ14"
 		(at 387.35 87.63 0)
 		(fields_autoplaced yes)
@@
 		)
 	)
-	(label "U47_DQ14"
+	(label "UO47_DQ14"
 		(at 317.5 87.63 0)
 		(fields_autoplaced yes)
@@
 		)
 	)
-	(label "U46_DQ14"
+	(label "UO46_DQ14"
 		(at 334.01 120.65 0)
 		(fields_autoplaced yes)
@@
 		)
 	)
-	(label "U46_DQ13"
+	(label "UO46_DQ13"
 		(at 334.01 123.19 0)
 		(fields_autoplaced yes)
@@
 		)
 	)
-	(label "U46_DQ15"
+	(label "UO46_DQ15"
 		(at 334.01 118.11 0)
 		(fields_autoplaced yes)
@@
 		)
 	)
-	(label "U47_DQ14"
+	(label "UO47_DQ14"
 		(at 334.01 130.81 0)
 		(fields_autoplaced yes)
@@
 		)
 	)
-	(label "U46_DQ15"
+	(label "UO46_DQ15"
 		(at 387.35 90.17 0)
 		(fields_autoplaced yes)
@@
 		)
 	)
-	(label "U47_DQ15"
+	(label "UO47_DQ15"
 		(at 317.5 90.17 0)
 		(fields_autoplaced yes)
@@
 		)
 	)
-	(label "U47_DQ15"
+	(label "UO47_DQ15"
 		(at 334.01 128.27 0)
 		(fields_autoplaced yes)
@@
 		)
 	)
-	(label "U46_DQ13"
+	(label "UO46_DQ13"
 		(at 387.35 85.09 0)
 		(fields_autoplaced yes)
@@
 		)
 	)
-	(label "U47_DQ13"
+	(label "UO47_DQ13"
 		(at 317.5 85.09 0)
 		(fields_autoplaced yes)
@@
 		(dnp no)
 		(fields_autoplaced yes)
-		(property "Reference" "U125"
+		(property "Reference" "UO125"
 			(at 298.1041 173.99 0)
 			(effects
@@
 			(project "ra9704"
 				(path "/24d3b4cf-2360-45fc-8c40-cedc8afdf9e1/4c59c4b7-e848-4b36-8bfe-90f55a1ec475"
-					(reference "U125")
+					(reference "UO125")
 					(unit 1)
 				)
@@
 		(on_board yes)
 		(dnp no)
-		(property "Reference" "RA41"
+		(property "Reference" "RA041"
 			(at 349.504 113.284 90)
 			(effects
@@
 			(project "ra9704"
 				(path "/24d3b4cf-2360-45fc-8c40-cedc8afdf9e1/4c59c4b7-e848-4b36-8bfe-90f55a1ec475"
-					(reference "RA41")
+					(reference "RA041")
 					(unit 1)
 				)
@@
 		(dnp no)
 		(fields_autoplaced yes)
-		(property "Reference" "U126"
+		(property "Reference" "UO126"
 			(at 362.8741 173.99 0)
 			(effects
@@
 			(project "ra9704"
 				(path "/24d3b4cf-2360-45fc-8c40-cedc8afdf9e1/4c59c4b7-e848-4b36-8bfe-90f55a1ec475"
-					(reference "U126")
+					(reference "UO126")
 					(unit 1)
 				)
@@
 		(on_board yes)
 		(dnp no)
-		(property "Reference" "U47"
+		(property "Reference" "UO47"
 			(at 308.61 44.704 0)
 			(effects
@@
 			(project "ra9704"
 				(path "/24d3b4cf-2360-45fc-8c40-cedc8afdf9e1/4c59c4b7-e848-4b36-8bfe-90f55a1ec475"
-					(reference "U47")
+					(reference "UO47")
 					(unit 1)
 				)
@@
 		(on_board yes)
 		(dnp no)
-		(property "Reference" "U46"
+		(property "Reference" "UO46"
 			(at 377.952 44.704 0)
 			(effects
@@
 			(project "ra9704"
 				(path "/24d3b4cf-2360-45fc-8c40-cedc8afdf9e1/4c59c4b7-e848-4b36-8bfe-90f55a1ec475"
-					(reference "U46")
+					(reference "UO46")
 					(unit 1)
 				)
@@
 		(on_board yes)
 		(dnp no)
-		(property "Reference" "U42"
-			(at 124.968 133.35 0)
+		(property "Reference" "UO42"
+			(at 117.348 132.842 0)
 			(effects
 				(font
@@
 			(project "ra9704"
 				(path "/24d3b4cf-2360-45fc-8c40-cedc8afdf9e1/4c59c4b7-e848-4b36-8bfe-90f55a1ec475"
-					(reference "U42")
+					(reference "UO42")
 					(unit 1)
 				)
