File: Toaplan2/Raizing/RA9704/ra9704-kicad/main-ic-bus-mgmt.kicad_sch (KiCad schematic)
At the start: 19 parts, among them U114 E68DEC2 (GAL16V8), U117 PST518A, U118 74AC14, U19 MAIN_IF2 (MACH211), U48 AFBK_CT2 (MACH211), U623 VVEC2_3A (MACH211), U624 A11235, X11 32 MHz, X61 27 MHz

Commit message: feature(ra9704): rev 002
Parts:
- removed C1: 23 mF, ra9704:C_Disc_D5.0mm_W2.5mm_P5.00mm, symbol ra9704:C_Disc
- removed C61, C62, C63: 101 pF, ra9704:C_Disc_D5.0mm_W2.5mm_P5.00mm, symbol ra9704:C_Disc
- removed JP61: Jumper_2_Open, ra9704:PinHeader_2x01_P2.54mm_Vertical, symbol ra9704:Jumper_2_Open
- removed R61: 220Ω, ra9704:R_Axial_DIN0204_L3.6mm_D1.6mm_P5.08mm_Horizontal, symbol ra9704:R
- removed unit 3 of U118
- removed U623: VVEC2_3A (MACH211), ra9704:PLCC-44, symbol ra9704:MACH211
- removed U624: A11235, ra9704:PLCC-68, symbol ra9704:A11235
- removed X61: 27 MHz, Oscillator:Oscillator_DIP-14, symbol ra9704:Oscillator
Connections:
- no-connect marks 28 -> 22
Other:
- note removed: "A tantalum 23 mF is jumped here"
- note removed: "TVRMCTL7"
- note removed: "UNDER CONSTRUCTION"
- moved on the sheet: C11, D119, R13, R14, U114, U117, U118A, U118G, U19, U48, X11
