File: Toaplan2/Raizing/RA9704/ra9704-kicad/main-ram-and-rom.kicad_sch (KiCad schematic)
At the start: 7 parts, among them U21 PRG2 (27C040), U22 PRG0 (27C040), U23 PRG1 (27C040), U24 PRG3 (27C040), U25 CY7C199, U26 CY7C199

Commit message: feature(ra9704): rev 002
Other:
- moved on the sheet: U21, U22, U23, U24, U25, U26
