File: Toaplan2/Raizing/RA9704/ra9704-kicad/main-ram-and-rom.kicad_sch (KiCad schematic)
At the start: 7 parts, among them U21 PRG2 (27C040), U22 PRG0 (27C040), U23 PRG1 (27C040), U24 PRG3 (27C040), U25 CY7C199, U26 CY7C199

Commit message: fix(ra9704): Add Os as a proxy for 0s in all reference designators
RA9704 has reference designators such that each number has a preceding zero (e.g. RA076, U074, etc.). This causes a bug in KiCAD.

This is 'fixed' by using the 'O' (the letter 'Oh') character instead.

For more info, see the following issue on the KiCAD Gitlab repo

https://gitlab.com/kicad/code/kicad/-/issues/19229
Parts:
- renumbered JP21 to JPO21, U21 to UO21, U22 to UO22, U23 to UO23, U24 to UO24, U25 to UO25, U26 to UO26
Changed lines of the file:
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@@
 		(dnp no)
 		(fields_autoplaced yes)
-		(property "Reference" "U23"
+		(property "Reference" "UO23"
 			(at 80.9341 157.48 0)
 			(effects
@@
 			(project "ra9704"
 				(path "/24d3b4cf-2360-45fc-8c40-cedc8afdf9e1/91f305cd-cca6-4908-92ee-ec1491f84c70"
-					(reference "U23")
+					(reference "UO23")
 					(unit 1)
 				)
@@
 		(dnp no)
 		(fields_autoplaced yes)
-		(property "Reference" "U25"
+		(property "Reference" "UO25"
 			(at 79.6641 17.78 0)
 			(effects
@@
 			(project "ra9704"
 				(path "/24d3b4cf-2360-45fc-8c40-cedc8afdf9e1/91f305cd-cca6-4908-92ee-ec1491f84c70"
-					(reference "U25")
+					(reference "UO25")
 					(unit 1)
 				)
@@
 		(dnp no)
 		(fields_autoplaced yes)
-		(property "Reference" "U26"
+		(property "Reference" "UO26"
 			(at 148.2441 17.78 0)
 			(effects
@@
 			(project "ra9704"
 				(path "/24d3b4cf-2360-45fc-8c40-cedc8afdf9e1/91f305cd-cca6-4908-92ee-ec1491f84c70"
-					(reference "U26")
+					(reference "UO26")
 					(unit 1)
 				)
@@
 		(dnp no)
 		(fields_autoplaced yes)
-		(property "Reference" "U21"
+		(property "Reference" "UO21"
 			(at 80.9341 78.74 0)
 			(effects
@@
 			(project "ra9704"
 				(path "/24d3b4cf-2360-45fc-8c40-cedc8afdf9e1/91f305cd-cca6-4908-92ee-ec1491f84c70"
-					(reference "U21")
+					(reference "UO21")
 					(unit 1)
 				)
@@
 		(dnp no)
 		(fields_autoplaced yes)
-		(property "Reference" "U22"
+		(property "Reference" "UO22"
 			(at 148.2441 80.01 0)
 			(effects
@@
 			(project "ra9704"
 				(path "/24d3b4cf-2360-45fc-8c40-cedc8afdf9e1/91f305cd-cca6-4908-92ee-ec1491f84c70"
-					(reference "U22")
+					(reference "UO22")
 					(unit 1)
 				)
@@
 		(on_board yes)
 		(dnp no)
-		(property "Reference" "JP21"
+		(property "Reference" "JPO21"
 			(at 50.8 240.284 0)
 			(effects
@@
 			(project "ra9704"
 				(path "/24d3b4cf-2360-45fc-8c40-cedc8afdf9e1/91f305cd-cca6-4908-92ee-ec1491f84c70"
-					(reference "JP21")
+					(reference "JPO21")
 					(unit 1)
 				)
@@
 		(dnp no)
 		(fields_autoplaced yes)
-		(property "Reference" "U24"
+		(property "Reference" "UO24"
 			(at 148.2441 157.48 0)
 			(effects
@@
 			(project "ra9704"
 				(path "/24d3b4cf-2360-45fc-8c40-cedc8afdf9e1/91f305cd-cca6-4908-92ee-ec1491f84c70"
-					(reference "U24")
-					(unit 1)
-				)
+					(reference "UO24")
+					(unit 1)
+				)
