File: Toaplan2/Raizing/RA9704/ra9704-kicad/ra9704.kicad_sch (KiCad schematic)
At the start: 0 parts

Commit message: feature(ra9704): rev 002
Other:
- removed sheet Video RAM
- added sheet Video RAM and Bus Mgmt (video-ram-and-bus-mgmt.kicad_sch)
- sheet Audio DAC, SFX Roms ports: added SBUS_A[0..15], SFX1_A[0..18], SFX2_A[0..18], SFX2_VPP; removed SBUS_A0, SFX1_A[0..7], SFX2_A[0..7]
- sheet GCU and GCU_V RAM ports: added GCU_OSCCLK; removed none
- sheet Main IC and Bus Mgmt ports: added COIN_DOUT_CLK, CTRLS1_BUS_~{OE}, CTRLS2_BUS_~{OE}, CTRLS3_BUS_~{OE}, GCU_ACK, GCU_CS, GCU_D[0..15], GCU_FRA[0..20], GCU_RS0, GROM-42, GROM-A18, GROM-~{BYTE}V_{PP}, GROM-~{G}0, GROM-~{G}1, GROM-~{G}2, MAINIF2_SUBDEC1_CTL, MAINIF2_TVRMCTL7_CTL, MBUS_A[0..23], MBUS_D[0..15], MCPU_CLK, MCPU_FC0, MCPU_FC1, MCPU_FC2, MCPU_GCU_D_CE, MCPU_MUSROM_~{CE}, MCPU_R/~{W}, MCPU_~{AS}, MCPU_~{BGACK}, MCPU_~{DTACK}, MCPU_~{HALT}, MCPU_~{LDS}, MCPU_~{RESET}, MCPU_~{UDS}, MCPU_~{VPA}, MRAM_LSB_~{WE}, MRAM_MSB_~{WE}, MRAM_~{CE}, MROM_HIGH_~{CE}, MROM_LOW_~{CE}, PCM_EX23_CLK, SCPU_~{BUSRQ}, SCPU_~{CLK}, SCPU_~{RESET}, SUBDEC1_E68DEC2_CTL, VVEC23A_E68DEC2_CTL1, VVEC23A_E68DEC2_CTL2, YM2151_⌀M, ~{MBUS_A1}, ~{MBUS_A3}; removed none
- sheet Sound CPU and Memory ports: added none; removed M/SBUS_~{OE}
- sheet Sound IC and Bus Mgmt ports: added SBUS_A[0..15], SFX1_A[0..18], SFX2_A[0..18]; removed PCM_EXP1_CLK, SBUS_A[1..15], SFX1_A[8..18], SFX2_A[8..18]
- note removed: "UNDER CONSTRUCTION"
