File: Toaplan2/Raizing/RA9704/ra9704-kicad/sound-cpu-and-memory.kicad_sch (KiCad schematic)
At the start: 10 parts, among them U713 74HC244, U717 74HC367, U74 74HC244, U75 TMPZ84C00AP-8 (Z80), U77 27C020, U78 CY7C185

Commit message: feature(ra9704): rev 002
Connections:
- net M/SBUS_~{OE} is gone; now on net MCPU_SBUS_~{OE}: U713.1 (OEa), U713.19 (OEb), U74.1 (OEa), U74.19 (OEb)
