File: Toaplan2/Raizing/RA9704/ra9704-kicad/sound-ic-bus-mgmt.kicad_sch (KiCad schematic)
At the start: 5 parts, among them U715 PCM_EXP1 (GAL16V8), U716 PCM_EX23 (GAL16V8), U76 A101B

Commit message: feature(ra9704): rev 002
Other:
- note added: "PCM_EXP1_CLK is Unknown"
Changed lines of the file:
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@@
 	(title_block
 		(title "RA9704, Sound IC and Bus Mgmt")
-		(date "2024-12-29")
+		(date "2024-12-30")
 		(rev "002")
 		(company "Coin-Op Collection")
@@
 	(wire
 		(pts
+			(xy 36.83 60.96) (xy 52.07 60.96)
+		)
+		(stroke
+			(width 0)
+			(type default)
+		)
+	)
+	(wire
+		(pts
 			(xy 63.5 200.66) (xy 85.09 200.66)
 		)
@@
 		)
 	)
+	(text "PCM_EXP1_CLK is Unknown"
+		(exclude_from_sim no)
+		(at 283.21 116.84 0)
+		(effects
+			(font
+				(size 5 5)
+			)
+		)
+	)
 	(label "SFX1_A12"
 		(at 26.67 73.66 0)
@@
 		)
 	)
-	(label "SBUS_A[1..15]"
-		(at 24.13 222.25 0)
+	(label "SBUS_A[0..15]"
+		(at 105.41 119.38 0)
 		(fields_autoplaced yes)
 		(effects
@@
 		)
 	)
-	(label "SFX2_A[8..18]"
-		(at 121.92 106.68 0)
-		(fields_autoplaced yes)
-		(effects
-			(font
-				(size 1.27 1.27)
-			)
-			(justify left bottom)
+	(label "PCM_EXP1_CLK"
+		(at 52.07 60.96 180)
+		(fields_autoplaced yes)
+		(effects
+			(font
+				(size 1.27 1.27)
+			)
+			(justify right bottom)
 		)
 	)
@@
 		)
 	)
-	(label "SBUS_A[1..15]"
-		(at 104.14 119.38 0)
-		(fields_autoplaced yes)
-		(effects
-			(font
-				(size 1.27 1.27)
-			)
-			(justify left bottom)
-		)
-	)
 	(label "GCU_D7"
 		(at 142.24 208.28 0)
@@
 		)
 	)
-	(label "SBUS_A[1..15]"
-		(at 24.13 119.38 0)
-		(fields_autoplaced yes)
-		(effects
-			(font
-				(size 1.27 1.27)
-			)
-			(justify left bottom)
-		)
-	)
 	(label "SFX2_A10"
 		(at 124.46 67.31 0)
@@
 		)
 	)
+	(label "SFX2_A[0..18]"
+		(at 123.19 106.68 0)
+		(fields_autoplaced yes)
+		(effects
+			(font
+				(size 1.27 1.27)
+			)
+			(justify left bottom)
+		)
+	)
 	(label "GCU_D6"
 		(at 142.24 210.82 0)
@@
 		)
 	)
-	(label "SFX1_A[8..18]"
-		(at 154.94 209.55 0)
-		(fields_autoplaced yes)
-		(effects
-			(font
-				(size 1.27 1.27)
-			)
-			(justify left bottom)
-		)
-	)
 	(label "YM2151_D2"
 		(at 142.24 170.18 0)
@@
 		)
 	)
+	(label "SFX2_A[0..18]"
+		(at 156.21 198.12 0)
+		(fields_autoplaced yes)
+		(effects
+			(font
+				(size 1.27 1.27)
+			)
+			(justify left bottom)
+		)
+	)
 	(label "GCU_D[0..7]"
 		(at 44.45 125.73 0)
@@
 	)
 	(label "GCU_D[0..7]"
-		(at 121.92 125.73 0)
+		(at 123.19 125.73 0)
 		(fields_autoplaced yes)
 		(effects
@@
 		)
 	)
-	(label "SFX2_A[8..18]"
-		(at 154.94 198.12 0)
-		(fields_autoplaced yes)
-		(effects
-			(font
-				(size 1.27 1.27)
-			)
-			(justify left bottom)
-		)
-	)
 	(label "SBUS_A3"
 		(at 63.5 203.2 0)
@@
 		)
 	)
-	(label "SFX1_A[8..18]"
-		(at 24.13 113.03 0)
+	(label "SFX1_A[0..18]"
+		(at 25.4 113.03 0)
 		(fields_autoplaced yes)
 		(effects
@@
 		)
 	)
-	(label "SFX1_A[8..18]"
+	(label "SFX1_A[0..18]"
 		(at 179.07 181.61 90)
 		(fields_autoplaced yes)
@@
 		)
 	)
+	(label "SBUS_A[0..15]"
+		(at 25.4 222.25 0)
+		(fields_autoplaced yes)
+		(effects
+			(font
+				(size 1.27 1.27)
+			)
+			(justify left bottom)
+		)
+	)
 	(label "YM2151_D7"
 		(at 142.24 185.42 0)
@@
 		)
 	)
-	(label "SFX1_A[8..18]"
-		(at 121.92 113.03 0)
-		(fields_autoplaced yes)
-		(effects
-			(font
-				(size 1.27 1.27)
-			)
-			(justify left bottom)
-		)
-	)
-	(label "GCU_D[0..7]"
-		(at 153.67 222.25 0)
+	(label "SBUS_A[0..15]"
+		(at 25.4 119.38 0)
+		(fields_autoplaced yes)
+		(effects
+			(font
+				(size 1.27 1.27)
+			)
+			(justify left bottom)
+		)
+	)
+	(label "SFX1_A[0..18]"
+		(at 123.19 113.03 0)
 		(fields_autoplaced yes)
 		(effects
@@
 		)
 	)
-	(label "SFX2_A[8..18]"
+	(label "SFX2_A[0..18]"
 		(at 181.61 181.61 90)
+		(fields_autoplaced yes)
+		(effects
+			(font
+				(size 1.27 1.27)
+			)
+			(justify left bottom)
+		)
+	)
+	(label "GCU_D[0..7]"
+		(at 156.21 222.25 0)
 		(fields_autoplaced yes)
 		(effects
@@
 	(label "SBUS_A6"
 		(at 63.5 205.74 0)
+		(fields_autoplaced yes)
+		(effects
+			(font
+				(size 1.27 1.27)
+			)
+			(justify left bottom)
+		)
+	)
+	(label "SFX1_A[0..18]"
+		(at 156.21 209.55 0)
 		(fields_autoplaced yes)
 		(effects
@@
 	)
 	(hierarchical_label "SCPU_~{RESET}"
-		(shape input)
+		(shape bidirectional)
 		(at 85.09 180.34 180)
 		(fields_autoplaced yes)
@@
 	)
 	(hierarchical_label "SFX2_VPP"
-		(shape input)
+		(shape output)
 		(at 130.81 187.96 0)
 		(fields_autoplaced yes)
@@
 	)
 	(hierarchical_label "SFX1_VPP"
-		(shape input)
+		(shape output)
 		(at 130.81 198.12 0)
 		(fields_autoplaced yes)
@@
 		)
 	)
-	(hierarchical_label "PCM_EXP1_CLK"
-		(shape input)
-		(at 52.07 60.96 180)
-		(fields_autoplaced yes)
-		(effects
-			(font
-				(size 1.27 1.27)
-			)
-			(justify right)
-		)
-	)
-	(hierarchical_label "SBUS_A[1..15]"
+	(hierarchical_label "SBUS_A[0..15]"
 		(shape bidirectional)
 		(at 185.42 119.38 0)
@@
 		)
 	)
-	(hierarchical_label "SFX2_A[8..18]"
+	(hierarchical_label "SFX2_A[0..18]"
 		(shape bidirectional)
 		(at 185.42 106.68 0)
@@
 		)
 	)
-	(hierarchical_label "SFX1_A[8..18]"
+	(hierarchical_label "SFX1_A[0..18]"
 		(shape bidirectional)
 		(at 185.42 113.03 0)
