File: Toaplan2/Raizing/RA9704/ra9704-kicad/gcu_f-rom-and-ram.kicad_sch (KiCad schematic)
At the start: 13 parts, among them J516 Conn_02x20_Odd_Even, J517 Conn_02x20_Odd_Even, U44 CY7C185, U45 CY7C185, U510 ROM-1, LH535A00D, U511 ROM-2, LH535A00D, U512 ROM-3, LH535A00D, U513 ROM-4, LH535A00D, U514 LH535A00D, U515 LH535A00D

Commit message: fix(ra9704): Add Os as a proxy for 0s in all reference designators
RA9704 has reference designators such that each number has a preceding zero (e.g. RA076, U074, etc.). This causes a bug in KiCAD.

This is 'fixed' by using the 'O' (the letter 'Oh') character instead.

For more info, see the following issue on the KiCAD Gitlab repo

https://gitlab.com/kicad/code/kicad/-/issues/19229
Parts:
- renumbered J516 to JO516, J517 to JO517, U44 to UO44, U45 to UO45, U510 to UO510, U511 to UO511, U512 to UO512, U513 to UO513, U514 to UO514, U515 to UO515
Changed lines of the file:
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@@
 		(dnp no)
 		(fields_autoplaced yes)
-		(property "Reference" "U512"
+		(property "Reference" "UO512"
 			(at 130.4641 49.53 0)
 			(effects
@@
 			(project "ra9704"
 				(path "/24d3b4cf-2360-45fc-8c40-cedc8afdf9e1/55e61f45-c86a-46c0-98af-469f87fdc572"
-					(reference "U512")
+					(reference "UO512")
 					(unit 1)
 				)
@@
 		(on_board yes)
 		(dnp yes)
-		(property "Reference" "J516"
+		(property "Reference" "JO516"
 			(at 296.672 43.434 0)
 			(effects
@@
 			(project "ra9704"
 				(path "/24d3b4cf-2360-45fc-8c40-cedc8afdf9e1/55e61f45-c86a-46c0-98af-469f87fdc572"
-					(reference "J516")
+					(reference "JO516")
 					(unit 1)
 				)
@@
 		(dnp yes)
 		(fields_autoplaced yes)
-		(property "Reference" "U514"
+		(property "Reference" "UO514"
 			(at 195.2341 50.8 0)
 			(effects
@@
 			(project "ra9704"
 				(path "/24d3b4cf-2360-45fc-8c40-cedc8afdf9e1/55e61f45-c86a-46c0-98af-469f87fdc572"
-					(reference "U514")
+					(reference "UO514")
 					(unit 1)
 				)
@@
 		(dnp no)
 		(fields_autoplaced yes)
-		(property "Reference" "U44"
+		(property "Reference" "UO44"
 			(at 286.6741 153.67 0)
 			(effects
@@
 			(project "ra9704"
 				(path "/24d3b4cf-2360-45fc-8c40-cedc8afdf9e1/55e61f45-c86a-46c0-98af-469f87fdc572"
-					(reference "U44")
+					(reference "UO44")
 					(unit 1)
 				)
@@
 		(dnp yes)
 		(fields_autoplaced yes)
-		(property "Reference" "U515"
+		(property "Reference" "UO515"
 			(at 195.2341 176.53 0)
 			(effects
@@
 			(project "ra9704"
 				(path "/24d3b4cf-2360-45fc-8c40-cedc8afdf9e1/55e61f45-c86a-46c0-98af-469f87fdc572"
-					(reference "U515")
+					(reference "UO515")
 					(unit 1)
 				)
@@
 		(dnp no)
 		(fields_autoplaced yes)
-		(property "Reference" "U513"
+		(property "Reference" "UO513"
 			(at 130.4641 176.53 0)
 			(effects
@@
 			(project "ra9704"
 				(path "/24d3b4cf-2360-45fc-8c40-cedc8afdf9e1/55e61f45-c86a-46c0-98af-469f87fdc572"
-					(reference "U513")
+					(reference "UO513")
 					(unit 1)
 				)
@@
 		(dnp no)
 		(fields_autoplaced yes)
-		(property "Reference" "U510"
+		(property "Reference" "UO510"
 			(at 65.6941 49.53 0)
 			(effects
@@
 			(project "ra9704"
 				(path "/24d3b4cf-2360-45fc-8c40-cedc8afdf9e1/55e61f45-c86a-46c0-98af-469f87fdc572"
-					(reference "U510")
+					(reference "UO510")
 					(unit 1)
 				)
@@
 		(dnp no)
 		(fields_autoplaced yes)
-		(property "Reference" "U45"
+		(property "Reference" "UO45"
 			(at 357.7941 153.67 0)
 			(effects
@@
 			(project "ra9704"
 				(path "/24d3b4cf-2360-45fc-8c40-cedc8afdf9e1/55e61f45-c86a-46c0-98af-469f87fdc572"
-					(reference "U45")
+					(reference "UO45")
 					(unit 1)
 				)
@@
 		(on_board yes)
 		(dnp yes)
-		(property "Reference" "J517"
+		(property "Reference" "JO517"
 			(at 361.442 42.164 0)
 			(effects
@@
 			(project "ra9704"
 				(path "/24d3b4cf-2360-45fc-8c40-cedc8afdf9e1/55e61f45-c86a-46c0-98af-469f87fdc572"
-					(reference "J517")
+					(reference "JO517")
 					(unit 1)
 				)
@@
 		(dnp no)
 		(fields_autoplaced yes)
-		(property "Reference" "U511"
+		(property "Reference" "UO511"
 			(at 65.6941 176.53 0)
 			(effects
@@
 			(project "ra9704"
 				(path "/24d3b4cf-2360-45fc-8c40-cedc8afdf9e1/55e61f45-c86a-46c0-98af-469f87fdc572"
-					(reference "U511")
+					(reference "UO511")
 					(unit 1)
 				)
