File: Toaplan2/Raizing/RA9704/ra9704-kicad/main-cpu.kicad_sch (KiCad schematic)
At the start: 14 parts, among them U1 4.7kΩ, U11 TMP68HC000N-16 (M68K), U118 74AC14

Commit message: fix(ra9704): Add Os as a proxy for 0s in all reference designators
RA9704 has reference designators such that each number has a preceding zero (e.g. RA076, U074, etc.). This causes a bug in KiCAD.

This is 'fixed' by using the 'O' (the letter 'Oh') character instead.

For more info, see the following issue on the KiCAD Gitlab repo

https://gitlab.com/kicad/code/kicad/-/issues/19229
Parts:
- renumbered RA11 to RAO11, RA12 to RAO12, RA13 to RAO13, RA14 to RAO14, RA15 to RAO15, RA16 to RAO16, R11 to RO11, R12 to RO12, R15 to RO15, R16 to RO16, R17 to RO17, U11 to UO11, U118 to UO118
Changed lines of the file:
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@@
 		(dnp no)
 		(fields_autoplaced yes)
-		(property "Reference" "R17"
+		(property "Reference" "RO17"
 			(at 172.72 113.03 90)
 			(effects
@@
 			(project "ra9704"
 				(path "/24d3b4cf-2360-45fc-8c40-cedc8afdf9e1/bee75b16-e87f-4085-aaf6-73b306652624"
-					(reference "R17")
+					(reference "RO17")
 					(unit 1)
 				)
@@
 		(on_board yes)
 		(dnp no)
-		(property "Reference" "RA15"
+		(property "Reference" "RAO15"
 			(at 142.24 141.224 90)
 			(effects
@@
 			(project "ra9704"
 				(path "/24d3b4cf-2360-45fc-8c40-cedc8afdf9e1/bee75b16-e87f-4085-aaf6-73b306652624"
-					(reference "RA15")
+					(reference "RAO15")
 					(unit 1)
 				)
@@
 		(dnp no)
 		(fields_autoplaced yes)
-		(property "Reference" "R15"
+		(property "Reference" "RO15"
 			(at 172.72 81.28 90)
 			(effects
@@
 			(project "ra9704"
 				(path "/24d3b4cf-2360-45fc-8c40-cedc8afdf9e1/bee75b16-e87f-4085-aaf6-73b306652624"
-					(reference "R15")
+					(reference "RO15")
 					(unit 1)
 				)
@@
 		(on_board yes)
 		(dnp no)
-		(property "Reference" "RA13"
+		(property "Reference" "RAO13"
 			(at 157.48 48.006 90)
 			(effects
@@
 			(project "ra9704"
 				(path "/24d3b4cf-2360-45fc-8c40-cedc8afdf9e1/bee75b16-e87f-4085-aaf6-73b306652624"
-					(reference "RA13")
+					(reference "RAO13")
 					(unit 1)
 				)
@@
 		(dnp no)
 		(fields_autoplaced yes)
-		(property "Reference" "R16"
+		(property "Reference" "RO16"
 			(at 172.72 96.52 90)
 			(effects
@@
 			(project "ra9704"
 				(path "/24d3b4cf-2360-45fc-8c40-cedc8afdf9e1/bee75b16-e87f-4085-aaf6-73b306652624"
-					(reference "R16")
+					(reference "RO16")
 					(unit 1)
 				)
@@
 		(dnp no)
 		(fields_autoplaced yes)
-		(property "Reference" "U118"
+		(property "Reference" "UO118"
 			(at 161.29 93.98 0)
 			(effects
@@
 			(project "ra9704"
 				(path "/24d3b4cf-2360-45fc-8c40-cedc8afdf9e1/bee75b16-e87f-4085-aaf6-73b306652624"
-					(reference "U118")
+					(reference "UO118")
 					(unit 5)
 				)
@@
 		(on_board yes)
 		(dnp no)
-		(property "Reference" "R11"
+		(property "Reference" "RO11"
 			(at 30.48 171.45 90)
 			(effects
@@
 			(project "ra9704"
 				(path "/24d3b4cf-2360-45fc-8c40-cedc8afdf9e1/bee75b16-e87f-4085-aaf6-73b306652624"
-					(reference "R11")
+					(reference "RO11")
 					(unit 1)
 				)
@@
 		(dnp no)
 		(fields_autoplaced yes)
-		(property "Reference" "U118"
+		(property "Reference" "UO118"
 			(at 160.02 78.74 0)
 			(effects
@@
 			(project "ra9704"
 				(path "/24d3b4cf-2360-45fc-8c40-cedc8afdf9e1/bee75b16-e87f-4085-aaf6-73b306652624"
-					(reference "U118")
+					(reference "UO118")
 					(unit 4)
 				)
@@
 		(dnp no)
 		(fields_autoplaced yes)
-		(property "Reference" "R12"
+		(property "Reference" "RO12"
 			(at 30.48 151.13 90)
 			(effects
@@
 			(project "ra9704"
 				(path "/24d3b4cf-2360-45fc-8c40-cedc8afdf9e1/bee75b16-e87f-4085-aaf6-73b306652624"
-					(reference "R12")
+					(reference "RO12")
 					(unit 1)
 				)
@@
 		(dnp no)
 		(fields_autoplaced yes)
-		(property "Reference" "U11"
+		(property "Reference" "UO11"
 			(at 82.2041 68.58 0)
 			(effects
@@
 			(project "ra9704"
 				(path "/24d3b4cf-2360-45fc-8c40-cedc8afdf9e1/bee75b16-e87f-4085-aaf6-73b306652624"
-					(reference "U11")
+					(reference "UO11")
 					(unit 1)
 				)
@@
 		(on_board yes)
 		(dnp no)
-		(property "Reference" "RA11"
+		(property "Reference" "RAO11"
 			(at 146.304 19.558 90)
 			(effects
@@
 			(project "ra9704"
 				(path "/24d3b4cf-2360-45fc-8c40-cedc8afdf9e1/bee75b16-e87f-4085-aaf6-73b306652624"
-					(reference "RA11")
+					(reference "RAO11")
 					(unit 1)
 				)
@@
 		(on_board yes)
 		(dnp no)
-		(property "Reference" "RA16"
+		(property "Reference" "RAO16"
 			(at 153.67 201.168 90)
 			(effects
@@
 			(project "ra9704"
 				(path "/24d3b4cf-2360-45fc-8c40-cedc8afdf9e1/bee75b16-e87f-4085-aaf6-73b306652624"
-					(reference "RA16")
+					(reference "RAO16")
 					(unit 1)
 				)
@@
 		(on_board yes)
 		(dnp no)
-		(property "Reference" "RA12"
+		(property "Reference" "RAO12"
 			(at 176.784 19.558 90)
 			(effects
@@
 			(project "ra9704"
 				(path "/24d3b4cf-2360-45fc-8c40-cedc8afdf9e1/bee75b16-e87f-4085-aaf6-73b306652624"
-					(reference "RA12")
+					(reference "RAO12")
 					(unit 1)
 				)
@@
 		(dnp no)
 		(fields_autoplaced yes)
-		(property "Reference" "U118"
+		(property "Reference" "UO118"
 			(at 161.29 110.49 0)
 			(effects
@@
 			(project "ra9704"
 				(path "/24d3b4cf-2360-45fc-8c40-cedc8afdf9e1/bee75b16-e87f-4085-aaf6-73b306652624"
-					(reference "U118")
+					(reference "UO118")
 					(unit 6)
 				)
@@
 		(on_board yes)
 		(dnp no)
-		(property "Reference" "RA14"
+		(property "Reference" "RAO14"
 			(at 171.196 141.478 90)
 			(effects
@@
 			(project "ra9704"
 				(path "/24d3b4cf-2360-45fc-8c40-cedc8afdf9e1/bee75b16-e87f-4085-aaf6-73b306652624"
-					(reference "RA14")
+					(reference "RAO14")
 					(unit 1)
 				)
@@
 		(dnp no)
 		(fields_autoplaced yes)
-		(property "Reference" "U118"
+		(property "Reference" "UO118"
 			(at 158.75 184.15 0)
 			(effects
@@
 			(project "ra9704"
 				(path "/24d3b4cf-2360-45fc-8c40-cedc8afdf9e1/bee75b16-e87f-4085-aaf6-73b306652624"
-					(reference "U118")
+					(reference "UO118")
 					(unit 2)
 				)
