File: Toaplan2/Raizing/RA9704/ra9704-kicad/jamma.kicad_sch (KiCad schematic)
At the start: 5 parts

Commit message: fix(ra9704): Add Os as a proxy for 0s in all reference designators
RA9704 has reference designators such that each number has a preceding zero (e.g. RA076, U074, etc.). This causes a bug in KiCAD.

This is 'fixed' by using the 'O' (the letter 'Oh') character instead.

For more info, see the following issue on the KiCAD Gitlab repo

https://gitlab.com/kicad/code/kicad/-/issues/19229
Parts:
- renumbered C31 to CO31, C32 to CO32, C813 to CO813, C814 to CO814
Changed lines of the file:
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@@
 		(dnp no)
 		(fields_autoplaced yes)
-		(property "Reference" "C814"
+		(property "Reference" "CO814"
 			(at 140.97 99.6949 0)
 			(effects
@@
 			(project "ra9704"
 				(path "/24d3b4cf-2360-45fc-8c40-cedc8afdf9e1/4dc44d00-4a88-41ca-8358-795d7f7cc7d5"
-					(reference "C814")
+					(reference "CO814")
 					(unit 1)
 				)
@@
 		(dnp no)
 		(fields_autoplaced yes)
-		(property "Reference" "C31"
+		(property "Reference" "CO31"
 			(at 52.07 98.4249 0)
 			(effects
@@
 			(project "ra9704"
 				(path "/24d3b4cf-2360-45fc-8c40-cedc8afdf9e1/4dc44d00-4a88-41ca-8358-795d7f7cc7d5"
-					(reference "C31")
+					(reference "CO31")
 					(unit 1)
 				)
@@
 		(dnp no)
 		(fields_autoplaced yes)
-		(property "Reference" "C32"
+		(property "Reference" "CO32"
 			(at 69.85 98.4249 0)
 			(effects
@@
 			(project "ra9704"
 				(path "/24d3b4cf-2360-45fc-8c40-cedc8afdf9e1/4dc44d00-4a88-41ca-8358-795d7f7cc7d5"
-					(reference "C32")
+					(reference "CO32")
 					(unit 1)
 				)
@@
 		(dnp no)
 		(fields_autoplaced yes)
-		(property "Reference" "C813"
+		(property "Reference" "CO813"
 			(at 87.63 98.4249 0)
 			(effects
@@
 			(project "ra9704"
 				(path "/24d3b4cf-2360-45fc-8c40-cedc8afdf9e1/4dc44d00-4a88-41ca-8358-795d7f7cc7d5"
-					(reference "C813")
-					(unit 1)
-				)
+					(reference "CO813")
+					(unit 1)
+				)

Commit message: doc(ra9704): group 66 ceramic power caps and label on JAMMA page; replace uF with mu symbol
Parts:
- CO31, CO32, CO814: value 16V 470uF -> 16V 470μF
- CO813: value 25V 100uF -> 25V 100μF
Other:
- note added: "Four large capacitors to stabilize power plane voltages. Also, 66 unlabeled blue 1μF ceramic capacitors for this purpose are placed throughout."
- note removed: "Four large capacitors to stabilize power plane voltage"
Changed lines of the file:
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@@
 		)
 	)
-	(text "Four large capacitors to stabilize\npower plane voltage"
-		(exclude_from_sim no)
-		(at 64.516 89.408 0)
+	(text "Four large capacitors to stabilize power plane \nvoltages. Also, 66 unlabeled blue 1μF ceramic \ncapacitors for this purpose are placed throughout."
+		(exclude_from_sim no)
+		(at 68.326 90.424 0)
 		(effects
 			(font
@@
 			)
 		)
-		(property "Value" "16V 470uF"
+		(property "Value" "16V 470μF"
 			(at 140.97 102.2349 0)
 			(effects
@@
 			)
 		)
-		(property "Value" "16V 470uF"
+		(property "Value" "16V 470μF"
 			(at 52.07 100.9649 0)
 			(effects
@@
 			)
 		)
-		(property "Value" "16V 470uF"
+		(property "Value" "16V 470μF"
 			(at 69.85 100.9649 0)
 			(effects
@@
 			)
 		)
-		(property "Value" "25V 100uF"
+		(property "Value" "25V 100μF"
 			(at 87.63 100.9649 0)
 			(effects
